File: pi4-breakout.kicad_pcb (KiCad board)
At the start: 2 copper layers, 65 x 56 mm, 16 parts, among them J1 Raspberry_Pi, J2 I2C_0, J3 I2C_1, J4 I2C_2, J5 I2C_3, J6 UART, SW1 Power

Commit message: Export for fabrication
Other:
- board text added: "JLCJLCJLCJLC"
